Commit message: Update ADRC/PID

File: description/lidar.xacro (robot description, xacro)
@@ -48,5 +48,5 @@
                 <range>
                     <min>0.2</min>
-                    <max>12</max>
+                    <max>3</max>
                 </range>
             </lidar>

File: description/twbot.xacro (robot description, xacro)
@@ -85,5 +85,5 @@
     <axis xyz="0 1 0" />
     <dynamics damping="0.5" friction="0.01"/> <!--hadi friction t3 joint ( tsma moteur mchi les roues )-->
-    <limit effort="100.0" velocity="100.0"/>
+    <limit effort="50.0" velocity="20.0"/>
 </joint>
 <!--Left_Wheel_link-->
@@ -119,5 +119,5 @@
     <axis xyz="0 1 0" />
     <dynamics damping="0.5" friction="0.01"/>
-    <limit effort="100.0" velocity="100.0"/>
+    <limit effort="50.0" velocity="20.0"/>
 </joint>
 </robot>
